File: float_pcb.kicad_pcb (KiCad board)
At the start: 2 copper layers, 71 x 41.5 mm, 46 parts, among them J1 BR Switch, J2 5V, J3 USB_C, J4 Conn_01x02, J5 BR_DEPTH_SENSOR, J6 BR Light, J7 Batt, Q1 AO3400A, SW2 SW_Push, SW3 ENABLE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

Commit message: First Version
Parts:
- removed J4: Conn_01x02, Connector_PinHeader_2.54mm:PinHeader_1x02_P2.54mm_Vertical
- removed R18, R19: R, Resistor_SMD:R_0805_2012Metric
- removed VR1, VR2: TPSM863252RDXR, TPSM863252RDXR:VREG_TPSM863252RDXR
- added C13: 100n, Capacitor_SMD:C_0805_2012Metric, F.Cu at (136.0, 66.8)
- added C14: 1u, Capacitor_SMD:C_0805_2012Metric, F.Cu at (136.0, 71.2)
- added G***: LOGO, LOGO, F.Cu at (107.2, 66.8)
- added H1: MH, MountingHole:MountingHole_2.2mm_M2, F.Cu at (95.5, 65.5)
- added H2: MH, MountingHole:MountingHole_2.2mm_M2, F.Cu at (115.8, 100.2)
- added H3: MH, MountingHole:MountingHole_2.2mm_M2, F.Cu at (158.0, 64.5)
- added H4: MH, MountingHole:MountingHole_2.2mm_M2, F.Cu at (146.5, 100.5)
- added J8: Conn_01x04, Connector_PinHeader_2.54mm:PinHeader_1x04_P2.54mm_Vertical, F.Cu at (157.8, 76.6)
- added U1: TPSM863252, float_pcb_footprints:TPSM86325x_RDX0007A, F.Cu at (115.6, 89.1)
- added U2: TPSM863252, float_pcb_footprints:TPSM86325x_RDX0007A, F.Cu at (131.1, 97.6)
- C1, C6: value 10uF -> 10u
- C10, C5: value 33uF -> 33u
- C12: value 1uF -> 1u
- C2, C7: value 100nF -> 100n
- C3, C8: value 10nF -> 10n
- C4, C9: value 22pF -> 22p
- D3: value LED -> 5V_STAT
- ENABLE1: renamed from SW3; value ENABLE -> SW_Push
- J1, J2, J6: footprint Connector_JST:JST_VH_B2P-VH_1x02_P3.96mm_Vertical -> Connector_JST:JST_XH_B2B-XH-A_1x02_P2.50mm_Vertical
- J3: footprint Connector_USB:USB_C_Receptacle_HRO_TYPE-C-31-M-12 -> Connector_USB:USB_C_Receptacle_GCT_USB4105-xx-A_16P_TopMnt_Horizontal
- J5: value BR_DEPTH_SENSOR -> BR_DEPTH
- R1, R13: value 4.7kQ -> 4k7
- R10, R11: value 5.1kQ -> 5k1
- R12, R17, R3, R7: value 10kQ -> 10k
- R14: value 2.7kQ -> 2k7
- R15: value 650Q -> 650
- R16: value 1.5kQ -> 1k5; footprint LED_SMD:LED_0805_2012Metric -> Resistor_SMD:R_0805_2012Metric
- R2, R6: value 28.7kQ -> 28k7
- R4: value 135kQ -> 135k
- R5, R9: value 30kQ -> 30k
- R8: value 220kQ -> 220k
- moved R16 34.0 mm to (146.0, 95.8), turned to 90 degrees
- moved D3 33.1 mm to (146.0, 91.5), turned to -90 degrees
- moved R17 30.2 mm to (144.8, 86.0), turned to 90 degrees
- moved R15 27.2 mm to (135.5, 92.0), turned to 90 degrees
- moved D2 25.7 mm to (135.5, 88.0), turned to -90 degrees
- moved C12 25.1 mm to (132.2, 74.2), turned to -90 degrees
- moved R13 22.9 mm to (132.0, 83.5), turned to -90 degrees
- moved C1 22.1 mm to (95.5, 84.8), turned to 90 degrees
- moved R1 22.0 mm to (132.0, 79.2), turned to -90 degrees
- moved C9 21.1 mm to (136.0, 97.0)
- moved R12 20.5 mm to (128.5, 74.5)
- moved Q1 18.3 mm to (140.2, 86.0), turned to 180 degrees
- moved R3 18.3 mm to (105.2, 82.5), turned to 90 degrees
- moved C3 17.0 mm to (110.5, 89.0), turned to -90 degrees
- moved R2 16.9 mm to (105.2, 87.2), turned to 90 degrees
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- renumbered SW2 to BOOT1
Connections:
- BOOT1 pad 1: GND -> Net-(U3-IO0)
- BOOT1 pad 2: Net-(U3-IO0) -> GND
- C12 pad 1: GND -> Net-(U3-EN)
- C12 pad 2: Net-(U3-EN) -> GND
- C3 pad 1: Net-(VR1-EN) -> Net-(U1-EN)
- C8 pad 1: Net-(VR2-EN) -> Net-(U2-EN)
- J3 pad A4: unconnected-(J3-VBUS-PadA4)_2 -> /USB_VBUS_UNUSED
- J3 pad A9: unconnected-(J3-VBUS-PadA4)_1 -> /USB_VBUS_UNUSED
- J3 pad B4: unconnected-(J3-VBUS-PadA4)_3 -> /USB_VBUS_UNUSED
- J3 pad B9: unconnected-(J3-VBUS-PadA4) -> /USB_VBUS_UNUSED
- R11 pad 1: Net-(J3-CC2) -> GND
- R11 pad 2: GND -> Net-(J3-CC2)
- R2 pad 2: Net-(R2-Pad2) -> Net-(U1-EN)
- R3 pad 1: Net-(R2-Pad2) -> Net-(U1-EN)
- R6 pad 2: Net-(R6-Pad2) -> Net-(U2-EN)
- R7 pad 1: Net-(R6-Pad2) -> Net-(U2-EN)
- U3 pad 21: Net-(J4-Pin_2) -> unconnected-(U3-IO17-Pad21)
- U3 pad 22: Net-(J4-Pin_1) -> LIGHT
- U3 pad 35: unconnected-(U3-IO39-Pad35) -> Net-(J8-Pin_1)
- U3 pad 36: unconnected-(U3-IO40-Pad36) -> Net-(J8-Pin_2)
- U3 pad 37: LIGHT -> Net-(J8-Pin_3)
- U3 pad 38: unconnected-(U3-IO42-Pad38) -> Net-(J8-Pin_4)
Routing:
- net +3V3: track 0.00 -> 78.9 mm
- net Net-(U3-EN): track 0.00 -> 45.5 mm
- net +BATT: track 28.8 -> 60.7 mm
- net Net-(J6-Pin_2): track 0.00 -> 28.2 mm, vias 0 -> 2
- net Net-(U3-IO0): track 0.00 -> 25.9 mm, vias 0 -> 2
- net Net-(J2-Pin_1): track 0.00 -> 25.7 mm
- net /SDA: track 0.00 -> 19.3 mm, vias 0 -> 2
- net /SCL: track 0.00 -> 17.4 mm, vias 0 -> 2
- net Net-(U2-EN): track 0.00 -> 17.1 mm, vias 0 -> 2
- net Net-(U3-USB_D-): track 0.00 -> 17.1 mm
- net Net-(U1-EN): track 0.00 -> 16.3 mm
- net Net-(U1-FB): track 0.00 -> 15.3 mm, vias 0 -> 2
- net Net-(U2-FB): track 0.00 -> 15.2 mm, vias 0 -> 2
- net Net-(U3-USB_D+): track 0.00 -> 14.6 mm
- net GND: track 0.09 -> 13.8 mm, vias 0 -> 39
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- added copper zone on B.Cu, net GND
- added copper zone on F.Cu, net GND
Other:
- board size 71 x 41.5 mm -> 68.8 x 41.5 mm
- board text added: "FLOAT PCB V0 5/26"

Commit message: V2
Parts:
- removed G***: LOGO, LOGO
- removed H3, H4: MH, MountingHole:MountingHole_2.2mm_M2
- removed J2: 5V, Connector_JST:JST_XH_B2B-XH-A_1x02_P2.50mm_Vertical
- removed J8: Conn_01x04, Connector_PinHeader_2.54mm:PinHeader_1x04_P2.54mm_Vertical
- removed U3: ESP32-S3-MINI-1U, RF_Module:ESP32-S2-MINI-1U
- added J4: Conn_01x03, Connector_JST:JST_XH_B3B-XH-A_1x03_P2.50mm_Vertical, F.Cu at (142.2, 100.5)
- added J9: I2C, Connector_JST:JST_XH_B4B-XH-A_1x04_P2.50mm_Vertical, F.Cu at (123.8, 84.5)
- added LS1: SMT-0540-T-9-R, buzzer:XDCR_SMT-0540-T-9-R, F.Cu at (103.6, 76.5)
- added Q2: AO3400A, Package_TO_SOT_SMD:SOT-23, F.Cu at (109.3, 77.8)
- added R18: 4k7, Resistor_SMD:R_0603_1608Metric, F.Cu at (129.8, 84.5)
- added R19: 4k7, Resistor_SMD:R_0603_1608Metric, F.Cu at (129.8, 81.0)
- added R20: 10k, Resistor_SMD:R_0603_1608Metric, F.Cu at (118.8, 74.7)
- added U4: ESP32-S3-WROOM-1, RF_Module:ESP32-S3-WROOM-1U, F.Cu at (150.1, 81.5)
- C1, C10, C12, C13, C14, C2, C3, C4, C5, C6, C7, C8, C9: footprint Capacitor_SMD:C_0805_2012Metric -> Capacitor_SMD:C_0603_1608Metric
- D1: value BATT_STAT -> BATT; footprint LED_SMD:LED_0805_2012Metric -> LED_SMD:LED_0603_1608Metric
- D2: value LED -> 3V3; footprint LED_SMD:LED_0805_2012Metric -> LED_SMD:LED_0603_1608Metric
- D3: value 5V_STAT -> 5V; footprint LED_SMD:LED_0805_2012Metric -> LED_SMD:LED_0603_1608Metric
- J1: value BR Switch -> Switch
- J5: value BR_DEPTH -> I2C; footprint Connector_JST:JST_GH_BM04B-GHS-TBT_1x04-1MP_P1.25mm_Vertical -> Connector_JST:JST_XH_B4B-XH-A_1x04_P2.50mm_Vertical
- J6: value BR Light -> Light
- R1, R10, R11, R12, R13, R14, R15, R16, R17, R2, R3, R4, R5, R6, R7, R8, R9: footprint Resistor_SMD:R_0805_2012Metric -> Resistor_SMD:R_0603_1608Metric
- moved BOOT1 28.1 mm to (134.8, 91.1)
- moved R17 23.3 mm to (122.0, 91.0), turned to -90 degrees
- moved Q1 22.7 mm to (117.8, 89.2)
- moved H2 15.6 mm to (131.0, 96.8), turned to 0 degrees
- moved R9 14.6 mm to (127.0, 97.8)
- moved R8 14.6 mm to (127.0, 101.0)
- moved C5 14.1 mm to (117.5, 94.0)
- moved R1 13.3 mm to (118.8, 77.8)
- moved R13 13.3 mm to (118.8, 84.5)
- moved C9 13.3 mm to (122.8, 97.8)
- moved R5 13.0 mm to (113.2, 90.8)
- moved U2 12.9 mm to (118.3, 99.3)
- moved R11 12.8 mm to (149.0, 96.2)
- moved R4 12.6 mm to (113.2, 94.0)
- moved R10 12.5 mm to (149.0, 101.0)
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Connections:
- net /SCL renamed SCL1
- net /SDA renamed SDA1
- C1 pad 1: +BATT -> GND
- C1 pad 2: GND -> +BATT
- C7 pad 1: +BATT -> GND
- C7 pad 2: GND -> +BATT
- J1 pad 1: Net-(J1-Pin_1) -> +BATT
- J1 pad 2: +BATT -> Net-(J1-Pin_2)
- J6 pad 1: +3V3 -> Net-(J6-Pin_1)
- J6 pad 2: Net-(J6-Pin_2) -> +3V3
- J7 pad 2: Net-(J1-Pin_1) -> Net-(J1-Pin_2)
- Q1 pad 3: Net-(J6-Pin_2) -> Net-(J6-Pin_1)
Routing:
- net +3V3: track 78.9 -> 131.3 mm
- net BUZZER: track 0.00 -> 37.4 mm, vias 0 -> 4
- net Net-(J6-Pin_2): track 28.2 -> 0.00 mm, vias 2 -> 0
- net SCL2: track 0.00 -> 21.4 mm, vias 0 -> 2
- net Net-(J1-Pin_1): track 20.3 -> 0.00 mm
- net SDA2: track 0.00 -> 20.1 mm, vias 0 -> 2
- net Net-(U4-EN): track 45.5 -> 26.8 mm
- net Net-(J1-Pin_2): track 0.00 -> 17.6 mm
- net LIGHT: track 11.1 -> 25.5 mm, vias 0 -> 2
- net Net-(J6-Pin_1): track 0.00 -> 12.7 mm
- net +BATT: track 60.7 -> 48.3 mm
- net SCL1: track 17.4 -> 29.6 mm
- net SDA1: track 19.3 -> 31.0 mm
- net Net-(Q2-D): track 0.00 -> 8.14 mm
- net /USB_VBUS_UNUSED: track 6.96 -> 0.00 mm
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Other:
- board size 68.8 x 41.5 mm -> 68 x 32 mm
- board text added: "Dory V1"
- board text added: "Evan Kim '27"
- board text removed: "FLOAT PCB V0 5/26"

Commit message: V3
Parts:
- added H3: MH, MountingHole:MountingHole_2.2mm_M2, F.Cu at (206.7, 90.2)
- added J2: Conn_01x04, Connector_PinHeader_2.54mm:PinHeader_1x04_P2.54mm_Vertical, F.Cu at (240.0, 104.5)
- LS1: value SMT-0540-T-9-R -> AT-1127-ST-2-R; footprint buzzer:XDCR_SMT-0540-T-9-R -> buzzer:XDCR_AT-1127-ST-2-R
- moved LS1 147.3 mm to (246.2, 113.6)
- moved Q2 141.8 mm to (248.2, 106.0), turned to 0 degrees
- moved H1 138.1 mm to (226.2, 112.0)
- moved J1 131.6 mm to (226.2, 76.2), turned to 180 degrees
- moved R7 129.4 mm to (240.2, 76.2)
- moved C6 129.4 mm to (235.8, 76.2)
- moved C7 129.4 mm to (235.8, 72.9)
- moved D1 129.4 mm to (231.5, 76.2)
- moved R14 129.4 mm to (231.5, 72.9), turned to -90 degrees
- moved R6 129.4 mm to (240.2, 72.9)
- moved R8 124.6 mm to (250.5, 84.2), turned to -90 degrees
- moved R20 124.3 mm to (237.8, 110.8)
- moved C8 124.0 mm to (244.2, 76.2)
- moved C9 124.0 mm to (246.0, 84.2), turned to -90 degrees
- moved U2 119.9 mm to (237.2, 83.5)
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Connections:
- C10 pad 1: Net-(J4-Pin_2) -> GND
- C10 pad 2: GND -> Net-(J4-Pin_2)
- C12 pad 1: Net-(U4-EN) -> GND
- C12 pad 2: GND -> Net-(U4-EN)
- C4 pad 1: +3V3 -> Net-(U1-FB)
- C4 pad 2: Net-(U1-FB) -> +3V3
- C5 pad 1: +3V3 -> GND
- C5 pad 2: GND -> +3V3
- C9 pad 1: Net-(J4-Pin_2) -> Net-(U2-FB)
- C9 pad 2: Net-(U2-FB) -> Net-(J4-Pin_2)
- ENABLE1 pad 1: Net-(U4-EN) -> GND
- ENABLE1 pad 2: GND -> Net-(U4-EN)
- R11 pad 1: GND -> Net-(J3-CC2)
- R11 pad 2: Net-(J3-CC2) -> GND
- R14 pad 1: Net-(D1-A) -> +BATT
- R14 pad 2: +BATT -> Net-(D1-A)
- R15 pad 1: +3V3 -> Net-(D2-A)
- R15 pad 2: Net-(D2-A) -> +3V3
- R17 pad 1: GND -> LIGHT
- R17 pad 2: LIGHT -> GND
- R20 pad 1: GND -> BUZZER
- R20 pad 2: BUZZER -> GND
- R4 pad 1: +3V3 -> Net-(U1-FB)
- R4 pad 2: Net-(U1-FB) -> +3V3
- R5 pad 1: Net-(U1-FB) -> GND
- R5 pad 2: GND -> Net-(U1-FB)
- R8 pad 1: Net-(J4-Pin_2) -> Net-(U2-FB)
- R8 pad 2: Net-(U2-FB) -> Net-(J4-Pin_2)
- R9 pad 1: Net-(U2-FB) -> GND
- R9 pad 2: GND -> Net-(U2-FB)
- U4 pad 10: SDA1 -> unconnected-(U4-IO17-Pad10)
- U4 pad 11: SCL2 -> unconnected-(U4-IO18-Pad11)
- U4 pad 12: SDA2 -> unconnected-(U4-IO8-Pad12)
- U4 pad 16: SERVO -> SCL1
- U4 pad 17: unconnected-(U4-IO9-Pad17) -> SDA1
- U4 pad 24: unconnected-(U4-IO47-Pad24) -> SCL2
- U4 pad 25: unconnected-(U4-IO48-Pad25) -> SDA2
- U4 pad 26: unconnected-(U4-IO45-Pad26) -> BUZZER
- U4 pad 31: unconnected-(U4-IO38-Pad31) -> Net-(J2-Pin_1)
- U4 pad 32: unconnected-(U4-IO39-Pad32) -> Net-(J2-Pin_2)
- U4 pad 33: unconnected-(U4-IO40-Pad33) -> Net-(J2-Pin_3)
- U4 pad 34: unconnected-(U4-IO41-Pad34) -> Net-(J2-Pin_4)
- U4 pad 35: unconnected-(U4-IO42-Pad35) -> SERVO
- U4 pad 5: BUZZER -> unconnected-(U4-IO5-Pad5)
- U4 pad 9: SCL1 -> unconnected-(U4-IO16-Pad9)
Routing:
- net BUZZER: track 37.4 -> 16.1 mm, vias 4 -> 0
- net LIGHT: track 25.5 -> 7.10 mm, vias 2 -> 0
- net SDA1: track 31.0 -> 14.1 mm, vias 2 -> 0
- net SCL1: track 29.6 -> 14.8 mm, vias 2 -> 0
- net Net-(J1-Pin_2): track 17.6 -> 6.35 mm
- net Net-(U4-IO0): track 30.3 -> 20.6 mm, vias 2 -> 0
- net +BATT: track 48.3 -> 57.7 mm
- net SCL2: track 21.4 -> 13.1 mm, vias 2 -> 0
- net Net-(U4-EN): track 26.8 -> 18.7 mm
- net Net-(J6-Pin_1): track 12.7 -> 4.83 mm
- net /USB_VBUS_UNUSED: track 0.00 -> 6.68 mm
- net SDA2: track 20.1 -> 13.8 mm, vias 2 -> 0
- net SERVO: track 5.50 -> 11.9 mm
- net GND: track 9.41 -> 3.12 mm, vias 25 -> 42
- net Net-(J3-CC1): track 3.44 -> 9.42 mm
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Other:
- board size 68 x 32 mm -> 60 x 60 mm
- board text removed: "Evan Kim '27"

Commit message: Version 3
Before the big 4 layer migration
Parts:
- added G***: LOGO, LOGO, F.Cu at (227.0, 109.5)
- added G***: LOGO, LOGO, B.Cu at (227.3, 102.1)
- added TP1: 5V, TestPoint:TestPoint_Pad_D1.5mm, F.Cu at (250.0, 84.5)
- added TP2: 3V3, TestPoint:TestPoint_Pad_D1.5mm, F.Cu at (208.8, 118.3)
- added TP3: GND, TestPoint:TestPoint_Pad_D1.5mm, F.Cu at (237.8, 110.8)
- added TP4: BATT, TestPoint:TestPoint_Pad_D1.5mm, F.Cu at (230.0, 71.0)
- added U3: USBLC6-2SC6, Package_TO_SOT_SMD:SOT-23-6, F.Cu at (213.6, 105.3)
- C1, C10, C5, C6: footprint Capacitor_SMD:C_0603_1608Metric -> Capacitor_SMD:C_0805_2012Metric
- C14: value 1u -> 22u
- R14: value 2k7 -> 4k7
- R15: value 650 -> 1k
- R16: value 1k5 -> 2k2
- moved C3 15.4 mm to (203.2, 84.5), turned to 90 degrees
- moved C7 11.9 mm to (233.2, 84.5), turned to 90 degrees
- moved C5 7.54 mm to (219.8, 84.2)
- moved C4 7.45 mm to (224.0, 80.8)
- moved R20 6.95 mm to (243.8, 107.2)
- moved C2 6.68 mm to (211.5, 84.5), turned to 90 degrees
- moved C1 6.42 mm to (211.2, 81.0), turned to 90 degrees
- moved C6 5.55 mm to (233.0, 81.0), turned to 90 degrees
- moved R8 5.26 mm to (245.2, 84.0)
- moved R3 4.70 mm to (207.2, 81.2), turned to 90 degrees
- moved R14 4.01 mm to (233.8, 76.2), turned to 90 degrees
- moved D1 3.89 mm to (233.8, 73.0), turned to -90 degrees
- moved R15 3.81 mm to (228.0, 84.0)
- moved R5 3.81 mm to (219.5, 80.8)
- moved D2 3.79 mm to (228.0, 80.8)
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Connections:
- net /USB_VBUS_UNUSED renamed /VBUS
- C1 pad 1: GND -> +BATT
- C1 pad 2: +BATT -> GND
- C2 pad 1: +BATT -> GND
- C2 pad 2: GND -> +BATT
- C3 pad 1: Net-(U1-EN) -> GND
- C3 pad 2: GND -> Net-(U1-EN)
- C4 pad 1: Net-(U1-FB) -> +3V3
- C4 pad 2: +3V3 -> Net-(U1-FB)
- C9 pad 1: Net-(U2-FB) -> Net-(J4-Pin_2)
- C9 pad 2: Net-(J4-Pin_2) -> Net-(U2-FB)
- ENABLE1 pad 1: GND -> Net-(U4-EN)
- ENABLE1 pad 2: Net-(U4-EN) -> GND
- J3 pad A6: Net-(U4-USB_D+) -> Net-(J3-D+-PadA6)
- J3 pad A7: Net-(U4-USB_D-) -> Net-(J3-D--PadA7)
- J3 pad B6: Net-(U4-USB_D+) -> Net-(J3-D+-PadA6)
- J3 pad B7: Net-(U4-USB_D-) -> Net-(J3-D--PadA7)
- R10 pad 1: GND -> Net-(J3-CC1)
- R10 pad 2: Net-(J3-CC1) -> GND
- U4 pad 15: LIGHT -> unconnected-(U4-IO3-Pad15)
- U4 pad 16: SCL1 -> unconnected-(U4-IO46-Pad16)
- U4 pad 17: SDA1 -> LIGHT
- U4 pad 18: unconnected-(U4-IO10-Pad18) -> SCL1
- U4 pad 19: unconnected-(U4-IO11-Pad19) -> SDA1
- U4 pad 23: unconnected-(U4-IO21-Pad23) -> SCL2
- U4 pad 24: SCL2 -> SDA2
- U4 pad 25: SDA2 -> BUZZER
- U4 pad 26: BUZZER -> unconnected-(U4-IO45-Pad26)
Routing:
- net Net-(U4-USB_D+): track 19.8 -> 3.73 mm, vias 2 -> 0
- net Net-(U4-USB_D-): track 18.6 -> 3.48 mm, vias 2 -> 0
- net Net-(J3-D+-PadA6): track 0.00 -> 14.8 mm, vias 0 -> 2
- net Net-(J3-D--PadA7): track 0.00 -> 13.1 mm, vias 0 -> 2
- net /VBUS: track 6.68 -> 18.9 mm, vias 0 -> 2
- net +3V3: track 134.6 -> 142.9 mm
- net Net-(U1-FB): track 17.4 -> 12.3 mm
- net Net-(U2-FB): track 16.8 -> 11.9 mm, vias 2 -> 0
- net Net-(J4-Pin_2): track 25.9 -> 30.3 mm
- net +BATT: track 57.7 -> 61.7 mm
- net LIGHT: track 7.10 -> 10.3 mm
- net Net-(U1-EN): track 13.7 -> 15.7 mm
- net SCL2: track 13.1 -> 15.1 mm
- net SDA2: track 13.8 -> 15.6 mm
- net SDA1: track 14.1 -> 15.9 mm
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Other:
- board text added: "3V3"
- board text added: "5V"
- board text added: "DBG"
- board text added: "G"
- board text added: "GND"
- board text added: "NCSSM Morganton Evan Kim '27"
- board text added: "SCL"
- board text added: "SDA"
- board text added: "SIG"
- board text added: "Switch"
- board text added: "V"
- board text removed: "Dory V1"
